File: alim/carte_alimentation.kicad_pcb (KiCad board)
At the start: 2 copper layers, 33 parts, among them J11 Conn_01x02_Male, J12 Conn_01x02_Male, J21 Conn_01x02_Male, J22 Conn_01x02_Male, J31 Conn_01x02_Male, J32 Conn_01x02_Male, J40 Conn_01x02_Male, J42 Conn_01x02_Male, J43 Conn_01x02_Male, J44 Conn_01x02_Male, U1 LM2576T-5, U2 LM2576T-5, U3 LM2576T-5

Commit message: ajout led témoin alim
Parts:
- added D4: LED, LED_THT:LED_D3.0mm, F.Cu at (39.4, 127.0)
- added R4: R, Resistor_THT:R_Axial_DIN0411_L9.9mm_D3.6mm_P5.08mm_Vertical, F.Cu at (44.5, 124.5)
Routing:
- net Net-(C31-Pad1): track 39.3 -> 45.7 mm
- net Net-(D4-Pad2): track 0.00 -> 5.08 mm
Changed lines of the file:
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@@
     (thickness 1.6)
     (drawings 14)
-    (tracks 83)
+    (tracks 85)
     (zones 0)
-    (modules 33)
-    (nets 14)
+    (modules 35)
+    (nets 15)
   )
   (page A4)
@@
   )
   (setup
-    (last_trace_width 3)
+    (last_trace_width 1)
     (user_trace_width 1)
     (user_trace_width 1.8)
@@
   (net 12 "Net-(C22-Pad1)")
   (net 13 "Net-(C32-Pad1)")
+  (net 14 "Net-(D4-Pad2)")
   (net_class Default "This is the default net class."
     (clearance 0.2)
@@
     (add_net "Net-(D2-Pad1)")
     (add_net "Net-(D3-Pad1)")
+    (add_net "Net-(D4-Pad2)")
     (add_net "Net-(F41-Pad1)")
     (add_net "Net-(F41-Pad2)")
@@
     )
   )
+  (module LED_THT:LED_D3.0mm (layer F.Cu)
+    (at 39.37 127 270)
+    (descr "LED, diameter 3.0mm, 2 pins")
+    (tags "LED diameter 3.0mm 2 pins")
+    (fp_text reference D4 (at 1.27 -2.96 90) (layer F.SilkS)
+      (effects (font (size 1 1) (thickness 0.15)))
+    )
+    (fp_text value LED (at 1.27 2.96 90) (layer F.Fab)
+      (effects (font (size 1 1) (thickness 0.15)))
+    )
+    (fp_arc (start 1.27 0) (end -0.23 -1.16619) (angle 284.3) (layer F.Fab) (width 0.1))
+    (fp_arc (start 1.27 0) (end -0.29 -1.235516) (angle 108.8) (layer F.SilkS) (width 0.12))
+    (fp_arc (start 1.27 0) (end -0.29 1.235516) (angle -108.8) (layer F.SilkS) (width 0.12))
+    (fp_arc (start 1.27 0) (end 0.229039 -1.08) (angle 87.9) (layer F.SilkS) (width 0.12))
+    (fp_arc (start 1.27 0) (end 0.229039 1.08) (angle -87.9) (layer F.SilkS) (width 0.12))
+    (fp_circle (center 1.27 0) (end 2.77 0) (layer F.Fab) (width 0.1))
+    (fp_line (start -0.23 -1.16619) (end -0.23 1.16619) (layer F.Fab) (width 0.1))
+    (fp_line (start -0.29 -1.236) (end -0.29 -1.08) (layer F.SilkS) (width 0.12))
+    (fp_line (start -0.29 1.08) (end -0.29 1.236) (layer F.SilkS) (width 0.12))
+    (fp_line (start -1.15 -2.25) (end -1.15 2.25) (layer F.CrtYd) (width 0.05))
+    (fp_line (start -1.15 2.25) (end 3.7 2.25) (layer F.CrtYd) (width 0.05))
+    (fp_line (start 3.7 2.25) (end 3.7 -2.25) (layer F.CrtYd) (width 0.05))
+    (fp_line (start 3.7 -2.25) (end -1.15 -2.25) (layer F.CrtYd) (width 0.05))
+    (pad 1 thru_hole rect (at 0 0 270) (size 1.8 1.8) (drill 0.9) (layers *.Cu *.Mask)
+      (net 1 GND))
+    (pad 2 thru_hole circle (at 2.54 0 270) (size 1.8 1.8) (drill 0.9) (layers *.Cu *.Mask)
+      (net 14 "Net-(D4-Pad2)"))
+    (model ${KISYS3DMOD}/LED_THT.3dshapes/LED_D3.0mm.wrl
+      (at (xyz 0 0 0))
+      (scale (xyz 1 1 1))
+      (rotate (xyz 0 0 0))
+    )
+  )
+  (module Resistor_THT:R_Axial_DIN0411_L9.9mm_D3.6mm_P5.08mm_Vertical (layer F.Cu)
+    (at 44.45 124.46 270)
+    (descr "Resistor, Axial_DIN0411 series, Axial, Vertical, pin pitch=5.08mm, 1W, length*diameter=9.9*3.6mm^2")
+    (tags "Resistor Axial_DIN0411 series Axial Vertical pin pitch 5.08mm 1W length 9.9mm diameter 3.6mm")
+    (fp_text reference R4 (at 2.54 -2.92 90) (layer F.SilkS)
+      (effects (font (size 1 1) (thickness 0.15)))
+    )
+    (fp_text value R (at 2.54 2.92 90) (layer F.Fab)
+      (effects (font (size 1 1) (thickness 0.15)))
+    )
+    (fp_circle (center 0 0) (end 1.8 0) (layer F.Fab) (width 0.1))
+    (fp_circle (center 0 0) (end 1.92 0) (layer F.SilkS) (width 0.12))
+    (fp_line (start 0 0) (end 5.08 0) (layer F.Fab) (width 0.1))
+    (fp_line (start 1.92 0) (end 3.58 0) (layer F.SilkS) (width 0.12))
+    (fp_line (start -2.05 -2.05) (end -2.05 2.05) (layer F.CrtYd) (width 0.05))
+    (fp_line (start -2.05 2.05) (end 6.53 2.05) (layer F.CrtYd) (width 0.05))
+    (fp_line (start 6.53 2.05) (end 6.53 -2.05) (layer F.CrtYd) (width 0.05))
+    (fp_line (start 6.53 -2.05) (end -2.05 -2.05) (layer F.CrtYd) (width 0.05))
+    (fp_text user %R (at 2.54 -2.92 90) (layer F.Fab)
+      (effects (font (size 1 1) (thickness 0.15)))
+    )
+    (pad 1 thru_hole circle (at 0 0 270) (size 2.4 2.4) (drill 1.2) (layers *.Cu *.Mask)
+      (net 3 "Net-(C31-Pad1)"))
+    (pad 2 thru_hole oval (at 5.08 0 270) (size 2.4 2.4) (drill 1.2) (layers *.Cu *.Mask)
+      (net 14 "Net-(D4-Pad2)"))
+    (model ${KISYS3DMOD}/Resistor_THT.3dshapes/R_Axial_DIN0411_L9.9mm_D3.6mm_P5.08mm_Vertical.wrl
+      (at (xyz 0 0 0))
+      (scale (xyz 1 1 1))
+      (rotate (xyz 0 0 0))
+    )
+  )
   (gr_text Bot (at 111.76 130.81) (layer B.Cu)
     (effects (font (size 1.5 1.5) (thickness 0.3)))
@@
   (segment (start 44.45 110.525) (end 44.45 118.11) (width 3) (layer B.Cu) (net 3))
   (segment (start 44.485 110.49) (end 44.45 110.525) (width 3) (layer B.Cu) (net 3))
+  (segment (start 44.45 118.11) (end 44.45 124.46) (width 1) (layer B.Cu) (net 3))
   (segment (start 69.01 46.51) (end 69.01 49.706) (width 1.8) (layer B.Cu) (net 4))
   (segment (start 69.01 49.706) (end 73.914 54.61) (width 1.8) (layer B.Cu) (net 4))
@@
   (segment (start 104.14 113.03) (end 93.99 113.03) (width 1.8) (layer B.Cu) (net 13))
   (segment (start 130.81 113.03) (end 119.38 113.03) (width 1.8) (layer B.Cu) (net 13))
+  (segment (start 44.45 129.54) (end 39.37 129.54) (width 1) (layer B.Cu) (net 14))
   (zone (net 1) (net_name GND) (layer B.Cu) (hatch edge 0.508)
     (connect_pads (clearance 1))
