File: alim/carte_alimentation.kicad_pcb (KiCad board)
At the start: 2 copper layers, 35 parts, among them J11 Conn_01x02_Male, J12 Conn_01x02_Male, J21 Conn_01x02_Male, J22 Conn_01x02_Male, J31 Conn_01x02_Male, J32 Conn_01x02_Male, J40 Conn_01x02_Male, J42 Conn_01x02_Male, J43 Conn_01x02_Male, J44 Conn_01x02_Male, U1 LM2576T-5, U2 LM2576T-5, U3 LM2576T-5

Commit message: modif espacement et feedback
Parts:
- moved F41 2.54 mm to (41.9, 66.0)
- moved J44 2.54 mm to (39.4, 54.6)
- moved J31 2.54 mm to (133.3, 118.1)
- moved J40 1.27 mm to (39.4, 116.8)
- moved J12 1.27 mm to (133.3, 61.0)
Routing:
- net Net-(C32-Pad1): track 60.6 -> 73.3 mm
- net Net-(C22-Pad1): track 56.7 -> 65.5 mm
- net Net-(F41-Pad2): track 30.4 -> 31.5 mm
- net Net-(F41-Pad1): track 38.4 -> 39.3 mm
Changed lines of the file:
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@@
     (thickness 1.6)
     (drawings 14)
-    (tracks 85)
+    (tracks 87)
     (zones 0)
     (modules 35)
@@
   )
   (setup
-    (last_trace_width 0.25)
+    (last_trace_width 3)
     (user_trace_width 1)
     (user_trace_width 1.8)
@@
   )
   (module fusible:fusible_alim (layer F.Cu)
-    (at 44.45 66.04 180)
+    (at 41.91 66.04 180)
     (fp_text reference F41 (at -4.9 3.9) (layer F.SilkS)
       (effects (font (size 1 1) (thickness 0.15)))
@@
   )
   (module TerminalBlock:TerminalBlock_bornier-2_P5.08mm (layer F.Cu)
-    (at 132.08 60.96 90)
+    (at 133.35 60.96 90)
     (descr "simple 2-pin terminal block, pitch 5.08mm, revamped version of bornier2")
     (tags "terminal block bornier2")
@@
   )
   (module TerminalBlock:TerminalBlock_bornier-2_P5.08mm (layer F.Cu)
-    (at 130.81 118.11 90)
+    (at 133.35 118.11 90)
     (descr "simple 2-pin terminal block, pitch 5.08mm, revamped version of bornier2")
     (tags "terminal block bornier2")
@@
   )
   (module TerminalBlock:TerminalBlock_bornier-2_P5.08mm (layer F.Cu)
-    (at 39.37 118.11)
+    (at 39.37 116.84)
     (descr "simple 2-pin terminal block, pitch 5.08mm, revamped version of bornier2")
     (tags "terminal block bornier2")
@@
   )
   (module TerminalBlock:TerminalBlock_bornier-2_P5.08mm (layer F.Cu)
-    (at 39.37 52.07)
+    (at 39.37 54.61)
     (descr "simple 2-pin terminal block, pitch 5.08mm, revamped version of bornier2")
     (tags "terminal block bornier2")
@@
   )
   (via (at 39.37 110.49) (size 2) (drill 1) (layers F.Cu B.Cu) (net 1))
-  (via (at 39.37 91.44) (size 2) (drill 1) (layers F.Cu B.Cu) (net 1))
-  (via (at 39.37 59.69) (size 2) (drill 1) (layers F.Cu B.Cu) (net 1))
+  (via (at 39.37 92.71) (size 2) (drill 1) (layers F.Cu B.Cu) (net 1))
+  (via (at 39.37 60.96) (size 2) (drill 1) (layers F.Cu B.Cu) (net 1))
   (via (at 57.15 113.03) (size 2) (drill 1) (layers F.Cu B.Cu) (net 1))
   (via (at 64.77 85.09) (size 2) (drill 1) (layers F.Cu B.Cu) (net 1))
@@
   (segment (start 44.485 102.87) (end 59.69 102.87) (width 1.8) (layer B.Cu) (net 3))
   (segment (start 59.69 102.87) (end 68.58 102.87) (width 1.8) (layer B.Cu) (net 3))
-  (segment (start 44.45 110.525) (end 44.45 118.11) (width 3) (layer B.Cu) (net 3))
+  (segment (start 44.45 116.84) (end 44.45 124.46) (width 1) (layer B.Cu) (net 3))
+  (segment (start 44.45 110.525) (end 44.45 116.84) (width 3) (layer B.Cu) (net 3))
   (segment (start 44.485 110.49) (end 44.45 110.525) (width 3) (layer B.Cu) (net 3))
-  (segment (start 44.45 118.11) (end 44.45 124.46) (width 1) (layer B.Cu) (net 3))
   (segment (start 69.01 46.51) (end 69.01 49.706) (width 1.8) (layer B.Cu) (net 4))
   (segment (start 69.01 49.706) (end 73.914 54.61) (width 1.8) (layer B.Cu) (net 4))
@@
   (segment (start 70.28 108.38) (end 74.93 113.03) (width 1.8) (layer B.Cu) (net 6))
   (segment (start 78.38 113.03) (end 82.55 113.03) (width 1.8) (layer B.Cu) (net 6))
-  (segment (start 44.45 71.04) (end 44.45 66.04) (width 3) (layer B.Cu) (net 7))
-  (segment (start 44.45 40.64) (end 44.45 52.07) (width 3) (layer B.Cu) (net 7))
-  (segment (start 44.45 52.07) (end 44.45 66.04) (width 3) (layer B.Cu) (net 7))
-  (segment (start 44.45 81.04) (end 44.45 86.04) (width 3) (layer B.Cu) (net 8))
+  (segment (start 41.91 71.04) (end 41.91 66.04) (width 3) (layer B.Cu) (net 7))
+  (segment (start 44.45 63.5) (end 41.91 66.04) (width 3) (layer B.Cu) (net 7))
+  (segment (start 44.45 40.64) (end 44.45 63.5) (width 3) (layer B.Cu) (net 7))
   (segment (start 54.61 80.852) (end 54.61 85.852) (width 3) (layer B.Cu) (net 8))
   (segment (start 44.45 97.755) (end 44.485 97.79) (width 3) (layer B.Cu) (net 8))
-  (segment (start 44.45 86.04) (end 44.45 97.755) (width 3) (layer B.Cu) (net 8))
-  (segment (start 44.638 85.852) (end 44.45 86.04) (width 3) (layer B.Cu) (net 8))
   (segment (start 54.422 86.04) (end 54.61 85.852) (width 3) (layer B.Cu) (net 8))
   (segment (start 54.61 87.665) (end 44.485 97.79) (width 3) (layer B.Cu) (net 8))
   (segment (start 54.61 85.852) (end 54.61 87.665) (width 3) (layer B.Cu) (net 8))
+  (segment (start 44.485 97.79) (end 44.45 97.79) (width 3) (layer B.Cu) (net 8))
+  (segment (start 41.91 81.04) (end 41.91 86.04) (width 3) (layer B.Cu) (net 8))
+  (segment (start 44.485 97.79) (end 44.485 91.475) (width 3) (layer B.Cu) (net 8))
+  (segment (start 44.485 91.475) (end 44.45 91.44) (width 3) (layer B.Cu) (net 8))
+  (segment (start 44.45 88.58) (end 41.91 86.04) (width 3) (layer B.Cu) (net 8))
+  (segment (start 44.45 91.44) (end 44.45 88.58) (width 3) (layer B.Cu) (net 8))
   (segment (start 72.41 46.51) (end 75.43 49.53) (width 1) (layer B.Cu) (net 9))
   (segment (start 104.14 44.45) (end 97.79 44.45) (width 1) (layer B.Cu) (net 9))
@@
   (segment (start 121.84 85.17) (end 121.92 85.09) (width 1.8) (layer B.Cu) (net 12))
   (segment (start 109.22 85.17) (end 121.84 85.17) (width 1.8) (layer B.Cu) (net 12))
-  (segment (start 100.34 85.09) (end 95.26 80.01) (width 1) (layer B.Cu) (net 12))
-  (segment (start 95.26 80.01) (end 85.09 80.01) (width 1) (layer B.Cu) (net 12))
   (segment (start 81.3 75.72) (end 85.09 80.01) (width 1) (layer B.Cu) (net 12))
   (segment (start 85.09 80.01) (end 85.59 80.01) (width 1) (layer B.Cu) (net 12))
   (segment (start 121.92 85.09) (end 133.35 85.09) (width 1.8) (layer B.Cu) (net 12))
-  (segment (start 73.68 104.93) (end 76.7 107.95) (width 1) (layer B.Cu) (net 13))
+  (segment (start 104.14 80.01) (end 109.22 85.09) (width 1) (layer B.Cu) (net 12))
+  (segment (start 85.09 80.01) (end 104.14 80.01) (width 1) (layer B.Cu) (net 12))
   (segment (start 104.06 113.03) (end 104.14 113.11) (width 1.8) (layer B.Cu) (net 13))
   (segment (start 119.3 113.11) (end 119.38 113.03) (width 1.8) (layer B.Cu) (net 13))
   (segment (start 104.14 113.11) (end 119.3 113.11) (width 1.8) (layer B.Cu) (net 13))
-  (segment (start 92.190001 111.230001) (end 92.180001 111.230001) (width 1) (layer B.Cu) (net 13))
-  (segment (start 93.99 113.03) (end 92.190001 111.230001) (width 1) (layer B.Cu) (net 13))
-  (segment (start 88.9 107.95) (end 76.7 107.95) (width 1) (layer B.Cu) (net 13))
-  (segment (start 92.180001 111.230001) (end 88.9 107.95) (width 1) (layer B.Cu) (net 13))
   (segment (start 104.14 113.03) (end 93.99 113.03) (width 1.8) (layer B.Cu) (net 13))
   (segment (start 130.81 113.03) (end 119.38 113.03) (width 1.8) (layer B.Cu) (net 13))
+  (segment (start 99.06 107.95) (end 104.14 113.03) (width 1) (layer B.Cu) (net 13))
+  (segment (start 73.68 104.93) (end 76.7 107.95) (width 1) (layer B.Cu) (net 13))
+  (segment (start 76.7 107.95) (end 99.06 107.95) (width 1) (layer B.Cu) (net 13))
+  (segment (start 130.81 113.03) (end 133.35 113.03) (width 1.8) (layer B.Cu) (net 13))
   (segment (start 44.45 129.54) (end 39.37 129.54) (width 1) (layer B.Cu) (net 14))
   (zone (net 1) (net_name GND) (layer B.Cu) (hatch edge 0.508)
