File: alim/carte_alimentation.sch (KiCad schematic (older format))
At the start: 29 parts, among them J11 Conn_01x02_Male, J12 Conn_01x02_Male, J21 Conn_01x02_Male, J22 Conn_01x02_Male, J31 Conn_01x02_Male, J32 Conn_01x02_Male, J40 Conn_01x02_Male, J42 Conn_01x02_Male, J43 Conn_01x02_Male, J44 Conn_01x02_Male, U1 LM2576T-5, U2 LM2576T-5, U3 LM2576T-5

Commit message: ajout led témoin alim
Parts:
- added D4: LED, LED_THT:LED_D3.0mm, symbol Device:LED
- added R4: R, Resistor_THT:R_Axial_DIN0411_L9.9mm_D3.6mm_P5.08mm_Vertical, symbol Device:R
Connections:
- net GND: now also D4.1 (K)
- net at C31.1, J40.2 (Pin_2), J42.2 (Pin_2)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: now also R4.1
- new net: D4.2 (A), R4.2
Changed lines of the file:
@@
 Wire Wire Line
 	1500 2000 2450 2000
+$Comp
+L Device:LED D4
+U 1 1 5E198AD9
+P 1500 2650
+F 0 "D4" V 1539 2533 50  0000 R CNN
+F 1 "LED" V 1448 2533 50  0000 R CNN
+F 2 "LED_THT:LED_D3.0mm" H 1500 2650 50  0001 C CNN
+F 3 "~" H 1500 2650 50  0001 C CNN
+	1    1500 2650
+	0    -1   -1   0
+$EndComp
+$Comp
+L Device:R R4
+U 1 1 5E19B823
+P 1500 2350
+F 0 "R4" H 1570 2396 50  0000 L CNN
+F 1 "R" H 1570 2305 50  0000 L CNN
+F 2 "Resistor_THT:R_Axial_DIN0411_L9.9mm_D3.6mm_P5.08mm_Vertical" V 1430 2350 50  0001 C CNN
+F 3 "~" H 1500 2350 50  0001 C CNN
+	1    1500 2350
+	1    0    0    -1
+$EndComp
+Wire Wire Line
+	1500 2200 1500 2000
+Connection ~ 1500 2000
+$Comp
+L power:GND #PWR0125
+U 1 1 5E19D884
+P 1500 2800
+F 0 "#PWR0125" H 1500 2550 50  0001 C CNN
+F 1 "GND" H 1505 2627 50  0000 C CNN
+F 2 "" H 1500 2800 50  0001 C CNN
+F 3 "" H 1500 2800 50  0001 C CNN
+	1    1500 2800
+	1    0    0    -1
+$EndComp
 $EndSCHEMATC
